File: final.brd (EAGLE design)
At the start: 100 x 80 mm, 16 parts, among them IC1 7805TV, IC2 MEGA8-P, J1 POWER_JACKSLT

Commit message: design update
Parts:
- added R1, R2, R3, R4, R5, R6, R7, R8, R9: (no value), rcl:M0805
- moved C2 18.2 mm to (31.8, 48.3)
- moved J1 9.25 mm to (19.1, 44.5), turned to 270 degrees
- moved JP1 6.48 mm to (48.3, 16.5)
- moved C1 6.35 mm to (33.0, 30.5)
- moved Q1 5.08 mm to (44.5, 26.7)
- moved Q2 5.08 mm to (49.5, 26.7)
- moved Q3 5.08 mm to (54.6, 26.7)
- moved Q4 5.08 mm to (59.7, 26.7)
- moved Q5 5.08 mm to (64.8, 26.7)
- moved Q6 5.08 mm to (69.8, 26.7)
- moved Q7 5.08 mm to (74.9, 26.7)
- moved Q8 5.08 mm to (80.0, 26.7)
- moved Q9 5.08 mm to (85.1, 26.7)
- moved IC1 2.84 mm to (36.8, 44.5), turned to 90 degrees
Connections:
- net D0: now also R1.2
- net D1: now also R2.2
- net D2: now also R3.2
- net D3: now also R4.2
- net D4: now also R5.2
- net D5: now also R6.2
- net D6: now also R7.2
- net D7: now also R8.2
- net D8: now also R9.2
- net GND: now also R1.1, R2.1, R3.1, R4.1, R5.1, R6.1, R7.1, R8.1, R9.1
Routing:
- net GND: track 105.5 -> 0.00 mm
- net +5V: track 150.4 -> 47.3 mm
- net +12V: track 93.7 -> 64.2 mm
- net D2: track 6.35 -> 12.8 mm
- net D6: track 6.35 -> 12.8 mm
- net D4: track 8.45 -> 13.9 mm
- net D3: track 7.40 -> 12.8 mm
- net D1: track 7.40 -> 12.8 mm
- net D0: track 8.45 -> 13.9 mm
- net D8: track 8.45 -> 13.9 mm
- net D7: track 7.40 -> 12.8 mm
- net D5: track 7.40 -> 12.8 mm
- net N$13: track 12.8 -> 14.6 mm
- net N$14: track 15.3 -> 17.1 mm
- net N$12: track 10.3 -> 12.0 mm
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- added copper zone on layer 1, net GND
Other:
- board size 100 x 80 mm -> 78.4 x 52.1 mm
