File: final.sch (EAGLE design)
At the start: 16 parts, among them IC1 7805TV, IC2 MEGA8-P, J1 POWER_JACKSLT

Commit message: design update
Parts:
- added R1, R2, R3, R4, R5, R6, R7, R8, R9: (no value), rcl:R-EU_M0805
Connections:
- net D0: now also R1.2
- net D1: now also R2.2
- net D2: now also R3.2
- net D3: now also R4.2
- net D4: now also R5.2
- net D5: now also R6.2
- net D6: now also R7.2
- net D7: now also R8.2
- net D8: now also R9.2
- net GND: now also R1.1, R2.1, R3.1, R4.1, R5.1, R6.1, R7.1, R8.1, R9.1
Changed lines of the file:
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@@
 <part name="GND3" library="supply1" deviceset="GND" device=""/>
 <part name="IC2" library="atmel" deviceset="MEGA8-P" device=""/>
+<part name="R1" library="rcl" deviceset="R-EU_" device="M0805"/>
+<part name="R2" library="rcl" deviceset="R-EU_" device="M0805"/>
+<part name="R3" library="rcl" deviceset="R-EU_" device="M0805"/>
+<part name="R4" library="rcl" deviceset="R-EU_" device="M0805"/>
+<part name="R5" library="rcl" deviceset="R-EU_" device="M0805"/>
+<part name="R6" library="rcl" deviceset="R-EU_" device="M0805"/>
+<part name="R7" library="rcl" deviceset="R-EU_" device="M0805"/>
+<part name="R8" library="rcl" deviceset="R-EU_" device="M0805"/>
+<part name="R9" library="rcl" deviceset="R-EU_" device="M0805"/>
 </parts>
 <sheets>
@@
 <instance part="GND3" gate="1" x="40.64" y="48.26"/>
 <instance part="IC2" gate="G$1" x="43.18" y="91.44"/>
+<instance part="R1" gate="G$1" x="-12.7" y="-7.62" rot="R90"/>
+<instance part="R2" gate="G$1" x="0" y="-7.62" rot="R90"/>
+<instance part="R3" gate="G$1" x="12.7" y="-7.62" rot="R90"/>
+<instance part="R4" gate="G$1" x="25.4" y="-7.62" rot="R90"/>
+<instance part="R5" gate="G$1" x="38.1" y="-7.62" rot="R90"/>
+<instance part="R6" gate="G$1" x="50.8" y="-7.62" rot="R90"/>
+<instance part="R7" gate="G$1" x="66.04" y="-7.62" rot="R90"/>
+<instance part="R8" gate="G$1" x="78.74" y="-7.62" rot="R90"/>
+<instance part="R9" gate="G$1" x="93.98" y="-7.62" rot="R90"/>
 </instances>
 <busses>
@@
 <wire x1="-20.32" y1="-10.16" x2="-20.32" y2="-20.32" width="0.1524" layer="91"/>
 <pinref part="GND2" gate="1" pin="GND"/>
-<wire x1="-20.32" y1="-20.32" x2="-7.62" y2="-20.32" width="0.1524" layer="91"/>
+<wire x1="-20.32" y1="-20.32" x2="-12.7" y2="-20.32" width="0.1524" layer="91"/>
+<wire x1="-12.7" y1="-20.32" x2="-7.62" y2="-20.32" width="0.1524" layer="91"/>
 <wire x1="-7.62" y1="-20.32" x2="0" y2="-20.32" width="0.1524" layer="91"/>
 <wire x1="0" y1="-20.32" x2="0" y2="-33.02" width="0.1524" layer="91"/>
 <pinref part="Q9" gate="G$1" pin="D"/>
 <wire x1="83.82" y1="-10.16" x2="83.82" y2="-20.32" width="0.1524" layer="91"/>
-<wire x1="83.82" y1="-20.32" x2="71.12" y2="-20.32" width="0.1524" layer="91"/>
+<wire x1="83.82" y1="-20.32" x2="78.74" y2="-20.32" width="0.1524" layer="91"/>
 <junction x="0" y="-20.32"/>
 <pinref part="Q2" gate="G$1" pin="D"/>
-<wire x1="71.12" y1="-20.32" x2="58.42" y2="-20.32" width="0.1524" layer="91"/>
-<wire x1="58.42" y1="-20.32" x2="43.18" y2="-20.32" width="0.1524" layer="91"/>
-<wire x1="43.18" y1="-20.32" x2="30.48" y2="-20.32" width="0.1524" layer="91"/>
-<wire x1="30.48" y1="-20.32" x2="17.78" y2="-20.32" width="0.1524" layer="91"/>
-<wire x1="17.78" y1="-20.32" x2="5.08" y2="-20.32" width="0.1524" layer="91"/>
+<wire x1="78.74" y1="-20.32" x2="71.12" y2="-20.32" width="0.1524" layer="91"/>
+<wire x1="71.12" y1="-20.32" x2="66.04" y2="-20.32" width="0.1524" layer="91"/>
+<wire x1="66.04" y1="-20.32" x2="58.42" y2="-20.32" width="0.1524" layer="91"/>
+<wire x1="58.42" y1="-20.32" x2="50.8" y2="-20.32" width="0.1524" layer="91"/>
+<wire x1="50.8" y1="-20.32" x2="43.18" y2="-20.32" width="0.1524" layer="91"/>
+<wire x1="43.18" y1="-20.32" x2="38.1" y2="-20.32" width="0.1524" layer="91"/>
+<wire x1="38.1" y1="-20.32" x2="30.48" y2="-20.32" width="0.1524" layer="91"/>
+<wire x1="30.48" y1="-20.32" x2="25.4" y2="-20.32" width="0.1524" layer="91"/>
+<wire x1="25.4" y1="-20.32" x2="17.78" y2="-20.32" width="0.1524" layer="91"/>
+<wire x1="17.78" y1="-20.32" x2="12.7" y2="-20.32" width="0.1524" layer="91"/>
+<wire x1="12.7" y1="-20.32" x2="5.08" y2="-20.32" width="0.1524" layer="91"/>
 <wire x1="5.08" y1="-20.32" x2="0" y2="-20.32" width="0.1524" layer="91"/>
 <wire x1="-7.62" y1="-10.16" x2="-7.62" y2="-20.32" width="0.1524" layer="91"/>
@@
 <wire x1="71.12" y1="-10.16" x2="71.12" y2="-20.32" width="0.1524" layer="91"/>
 <junction x="71.12" y="-20.32"/>
+<pinref part="R1" gate="G$1" pin="1"/>
+<wire x1="-12.7" y1="-12.7" x2="-12.7" y2="-20.32" width="0.1524" layer="91"/>
+<junction x="-12.7" y="-20.32"/>
+<pinref part="R2" gate="G$1" pin="1"/>
+<wire x1="0" y1="-12.7" x2="0" y2="-20.32" width="0.1524" layer="91"/>
+<pinref part="R3" gate="G$1" pin="1"/>
+<wire x1="12.7" y1="-12.7" x2="12.7" y2="-20.32" width="0.1524" layer="91"/>
+<junction x="12.7" y="-20.32"/>
+<pinref part="R4" gate="G$1" pin="1"/>
+<wire x1="25.4" y1="-12.7" x2="25.4" y2="-20.32" width="0.1524" layer="91"/>
+<junction x="25.4" y="-20.32"/>
+<pinref part="R5" gate="G$1" pin="1"/>
+<wire x1="38.1" y1="-12.7" x2="38.1" y2="-20.32" width="0.1524" layer="91"/>
+<junction x="38.1" y="-20.32"/>
+<pinref part="R6" gate="G$1" pin="1"/>
+<wire x1="50.8" y1="-12.7" x2="50.8" y2="-20.32" width="0.1524" layer="91"/>
+<junction x="50.8" y="-20.32"/>
+<pinref part="R7" gate="G$1" pin="1"/>
+<wire x1="66.04" y1="-12.7" x2="66.04" y2="-20.32" width="0.1524" layer="91"/>
+<junction x="66.04" y="-20.32"/>
+<pinref part="R8" gate="G$1" pin="1"/>
+<wire x1="78.74" y1="-12.7" x2="78.74" y2="-20.32" width="0.1524" layer="91"/>
+<junction x="78.74" y="-20.32"/>
+<pinref part="R9" gate="G$1" pin="1"/>
+<wire x1="93.98" y1="-12.7" x2="93.98" y2="-20.32" width="0.1524" layer="91"/>
+<wire x1="93.98" y1="-20.32" x2="83.82" y2="-20.32" width="0.1524" layer="91"/>
+<junction x="83.82" y="-20.32"/>
 </segment>
 <segment>
@@
 <wire x1="-15.24" y1="-2.54" x2="-12.7" y2="-2.54" width="0.1524" layer="91"/>
 <label x="-15.24" y="-2.54" size="1.778" layer="95"/>
+<pinref part="R1" gate="G$1" pin="2"/>
 </segment>
 </net>
@@
 <wire x1="-2.54" y1="-2.54" x2="0" y2="-2.54" width="0.1524" layer="91"/>
 <label x="-2.54" y="-2.54" size="1.778" layer="95"/>
+<pinref part="R2" gate="G$1" pin="2"/>
 </segment>
 </net>
@@
 <wire x1="10.16" y1="-2.54" x2="12.7" y2="-2.54" width="0.1524" layer="91"/>
 <label x="10.16" y="-2.54" size="1.778" layer="95"/>
+<pinref part="R3" gate="G$1" pin="2"/>
 </segment>
 </net>
@@
 <wire x1="22.86" y1="-2.54" x2="25.4" y2="-2.54" width="0.1524" layer="91"/>
 <label x="22.86" y="-2.54" size="1.778" layer="95"/>
+<pinref part="R4" gate="G$1" pin="2"/>
 </segment>
 </net>
@@
 <wire x1="35.56" y1="-2.54" x2="38.1" y2="-2.54" width="0.1524" layer="91"/>
 <label x="35.56" y="-2.54" size="1.778" layer="95"/>
+<pinref part="R5" gate="G$1" pin="2"/>
 </segment>
 </net>
@@
 <wire x1="48.26" y1="-2.54" x2="50.8" y2="-2.54" width="0.1524" layer="91"/>
 <label x="48.26" y="-2.54" size="1.778" layer="95"/>
+<pinref part="R6" gate="G$1" pin="2"/>
 </segment>
 </net>
@@
 <wire x1="63.5" y1="-2.54" x2="66.04" y2="-2.54" width="0.1524" layer="91"/>
 <label x="63.5" y="-2.54" size="1.778" layer="95"/>
+<pinref part="R7" gate="G$1" pin="2"/>
 </segment>
 </net>
@@
 <wire x1="76.2" y1="-2.54" x2="78.74" y2="-2.54" width="0.1524" layer="91"/>
 <label x="76.2" y="-2.54" size="1.778" layer="95"/>
+<pinref part="R8" gate="G$1" pin="2"/>
 </segment>
 </net>
@@
 <wire x1="88.9" y1="-2.54" x2="93.98" y2="-2.54" width="0.1524" layer="91"/>
 <label x="88.9" y="-2.54" size="1.778" layer="95"/>
-</segment>
-</net>
+<pinref part="R9" gate="G$1" pin="2"/>
+</segment>
+</net>
